File: 4-in-1_ESC/4-in-1_ESC.kicad_pcb (KiCad board)
At the start: 2 copper layers, 75 parts, among them Q1 BSC070N10NS3G, Q10 BSC070N10NS3G, Q11 BSC070N10NS3G, Q12 BSC070N10NS3G, Q13 BSC070N10NS3G, Q14 BSC070N10NS3G, Q15 BSC070N10NS3G, Q16 BSC070N10NS3G, Q17 BSC070N10NS3G, Q18 BSC070N10NS3G, Q19 BSC070N10NS3G, Q2 BSC070N10NS3G, Q20 BSC070N10NS3G, Q21 BSC070N10NS3G, Q22 BSC070N10NS3G, Q23 BSC070N10NS3G, Q24 BSC070N10NS3G, Q3 BSC070N10NS3G, Q4 BSC070N10NS3G, Q5 BSC070N10NS3G, Q6 BSC070N10NS3G, Q7 BSC070N10NS3G, Q8 BSC070N10NS3G, Q9 BSC070N10NS3G, U10 LMR51610XDBVR, U11 AMS1117-3.3_C347222, U2 JSM6288Q, U3 JSM6288Q, U4 STM32G071GBU6, U5 JSM6288Q, U6 STM32G071GBU6, U7 STM32G071GBU6, U8 JSM6288Q, U9 STM32G071GBU6

Commit message: Schematic First Pass
Parts:
- removed R3: 5mΩ, Resistor_SMD:R_1206_3216Metric
- removed R4, R5: 10R, Resistor_SMD:R_0402_1005Metric
- removed R6: 10kΩ, Resistor_SMD:R_0402_1005Metric
- removed U8: JSM6288Q, easyeda_import:VQFN-24_L4.0-W4.0-P0.50-TL-EP2.7
- removed U9: STM32G071GBU6, easyeda_import:UFQFPN-28_L4.0-W4.0-P0.50-BL
- added C26: 10nF, Capacitor_SMD:C_0402_1005Metric, F.Cu at (140.1, 66.8)
- added C27: 10nF, Capacitor_SMD:C_0402_1005Metric, F.Cu at (140.1, 68.8)
- added C28: 10nF, Capacitor_SMD:C_0402_1005Metric, F.Cu at (140.1, 70.8)
- added C29: 4.7uF, Capacitor_SMD:C_0402_1005Metric, F.Cu at (140.1, 72.7)
- added C30: 4.7uF, Capacitor_SMD:C_0402_1005Metric, F.Cu at (140.1, 74.7)
- added C31: 4.7uF, Capacitor_SMD:C_0402_1005Metric, F.Cu at (143.0, 66.8)
- added C32: 10uF, Capacitor_SMD:C_0402_1005Metric, F.Cu at (143.0, 68.8)
- added C33: 100nF, Capacitor_SMD:C_0402_1005Metric, F.Cu at (143.0, 70.8)
- added C34: 10nF, Capacitor_SMD:C_0402_1005Metric, F.Cu at (140.1, 50.9)
- added C35: 10nF, Capacitor_SMD:C_0402_1005Metric, F.Cu at (140.1, 52.9)
- added C36: 10nF, Capacitor_SMD:C_0402_1005Metric, F.Cu at (140.1, 54.8)
- added C37: 4.7uF, Capacitor_SMD:C_0402_1005Metric, F.Cu at (140.1, 56.8)
- added C38: 4.7uF, Capacitor_SMD:C_0402_1005Metric, F.Cu at (140.1, 58.8)
- added C39: 4.7uF, Capacitor_SMD:C_0402_1005Metric, F.Cu at (143.0, 50.9)
- added C40: 10uF, Capacitor_SMD:C_0402_1005Metric, F.Cu at (143.0, 52.9)
- added C41: 100nF, Capacitor_SMD:C_0402_1005Metric, F.Cu at (143.0, 54.8)
- added C42: 10nF, Capacitor_SMD:C_0402_1005Metric, F.Cu at (122.8, 68.7)
- added C43: 10nF, Capacitor_SMD:C_0402_1005Metric, F.Cu at (122.8, 70.6)
- added C44: 10nF, Capacitor_SMD:C_0402_1005Metric, F.Cu at (122.8, 72.6)
- added C45: 4.7uF, Capacitor_SMD:C_0402_1005Metric, F.Cu at (122.8, 74.6)
- added C46: 4.7uF, Capacitor_SMD:C_0402_1005Metric, F.Cu at (122.8, 76.5)
- added C47: 4.7uF, Capacitor_SMD:C_0402_1005Metric, F.Cu at (125.6, 68.7)
- added C48: 10uF, Capacitor_SMD:C_0402_1005Metric, F.Cu at (125.6, 70.6)
- added C49: 100nF, Capacitor_SMD:C_0402_1005Metric, F.Cu at (125.6, 72.6)
- added C50: 10nF, Capacitor_SMD:C_0402_1005Metric, F.Cu at (140.1, 82.7)
- added C51: 10nF, Capacitor_SMD:C_0402_1005Metric, F.Cu at (140.1, 84.7)
- added C52: 10nF, Capacitor_SMD:C_0402_1005Metric, F.Cu at (140.1, 86.7)
- added C53: 4.7uF, Capacitor_SMD:C_0402_1005Metric, F.Cu at (140.1, 88.7)
- added C54: 100nF, Capacitor_SMD:C_0402_1005Metric, F.Cu at (143.0, 72.7)
- added C55: 100nF, Capacitor_SMD:C_0402_1005Metric, F.Cu at (114.0, 84.6)
- added C56: 100nF, Capacitor_SMD:C_0402_1005Metric, F.Cu at (143.0, 56.8)
- added C57: C_Small, Capacitor_SMD:C_0402_1005Metric, F.Cu at (114.0, 86.6)
- added C58: 4.7uF, Capacitor_SMD:C_0402_1005Metric, F.Cu at (140.1, 90.6)
- added C59: 4.7uF, Capacitor_SMD:C_0402_1005Metric, F.Cu at (143.0, 82.7)
- added C60: 10uF, Capacitor_SMD:C_0402_1005Metric, F.Cu at (143.0, 84.7)
- added C61: 100nF, Capacitor_SMD:C_0402_1005Metric, F.Cu at (143.0, 86.7)
- added C62: 100nF, Capacitor_SMD:C_0402_1005Metric, F.Cu at (125.6, 74.6)
- added C63: 100nF, Capacitor_SMD:C_0402_1005Metric, F.Cu at (147.9, 50.9)
- added C64: 100nF, Capacitor_SMD:C_0402_1005Metric, F.Cu at (143.0, 88.7)
- added C65: C_Small, Capacitor_SMD:C_0402_1005Metric, F.Cu at (147.9, 52.9)
- added C66: 100nF, Capacitor_SMD:C_0402_1005Metric, F.Cu at (114.0, 64.7)
- added C67: 4.7uF, Capacitor_SMD:C_0402_1005Metric, F.Cu at (143.0, 74.7)
- added C68: 4.7uF, Capacitor_SMD:C_0402_1005Metric, F.Cu at (143.0, 58.8)
- added C69: 4.7uF, Capacitor_SMD:C_0402_1005Metric, F.Cu at (125.6, 76.5)
- added C70: 4.7uF, Capacitor_SMD:C_0402_1005Metric, F.Cu at (143.0, 90.6)
- added C71: 100nF, Capacitor_SMD:C_0402_1005Metric, F.Cu at (147.9, 66.8)
- added C72: 100nF, Capacitor_SMD:C_0402_1005Metric, F.Cu at (114.0, 88.5)
- added C73: 100nF, Capacitor_SMD:C_0402_1005Metric, F.Cu at (147.9, 54.8)
- added C76: 100nF, Capacitor_SMD:C_0402_1005Metric, F.Cu at (121.8, 84.6)
- added C77: 2.2uF, Capacitor_SMD:C_0402_1005Metric, F.Cu at (121.8, 86.6)
- added C78: 10uF, Capacitor_SMD:C_0402_1005Metric, F.Cu at (121.8, 88.5)
- added C79: 22uF, Capacitor_SMD:C_0402_1005Metric, F.Cu at (121.8, 90.5)
- added C80: 4.7uF, Capacitor_SMD:C_0402_1005Metric, F.Cu at (147.9, 68.8)
- added C81: 100nF, Capacitor_SMD:C_0402_1005Metric, F.Cu at (147.9, 70.8)
- added C83: C_Small, Capacitor_SMD:C_0402_1005Metric, F.Cu at (147.9, 72.7)
- added C84: 4.7uF, Capacitor_SMD:C_0402_1005Metric, F.Cu at (114.0, 90.5)
- added C85: 100nF, Capacitor_SMD:C_0402_1005Metric, F.Cu at (147.9, 82.7)
- added C87: C_Small, Capacitor_SMD:C_0402_1005Metric, F.Cu at (147.9, 84.7)
- added C88: 100nF, Capacitor_SMD:C_0402_1005Metric, F.Cu at (147.9, 86.7)
- added C89: 4.7uF, Capacitor_SMD:C_0402_1005Metric, F.Cu at (147.9, 56.8)
- added C90: 4.7uF, Capacitor_SMD:C_0402_1005Metric, F.Cu at (147.9, 88.7)
- added CN1: SM10B-SRSS-TB, easyeda_import:CONN-SMD_10P-P1.00_SM10B-SRSS-TB-LF-SN, F.Cu at (119.5, 53.2)
- added CN2: SM07B-SRSS-TB, easyeda_import:CONN-SMD_SM07B-SRSS-TB, F.Cu at (118.0, 60.2)
- added FB10: 600Ω@100MHz, Inductor_SMD:L_0402_1005Metric, F.Cu at (150.8, 88.7)
- added FB11: 600Ω@100MHz, Inductor_SMD:L_0402_1005Metric, F.Cu at (114.1, 68.7)
- added FB12: 600Ω@100MHz, Inductor_SMD:L_0402_1005Metric, F.Cu at (131.4, 82.8)
- added FB5: 600Ω@100MHz, Inductor_SMD:L_0402_1005Metric, F.Cu at (116.9, 84.6)
- added FB6: 600Ω@100MHz, Inductor_SMD:L_0402_1005Metric, F.Cu at (150.8, 50.9)
- added FB7: 600Ω@100MHz, Inductor_SMD:L_0402_1005Metric, F.Cu at (131.4, 66.8)
- added FB8: 600Ω@100MHz, Inductor_SMD:L_0402_1005Metric, F.Cu at (131.4, 50.9)
- added FB9: 600Ω@100MHz, Inductor_SMD:L_0402_1005Metric, F.Cu at (150.8, 72.7)
- added R10: 130k, Resistor_SMD:R_0402_1005Metric, F.Cu at (131.4, 74.8)
- added R11: 10k, Resistor_SMD:R_0402_1005Metric, F.Cu at (131.4, 76.8)
- added R12: 1k, Resistor_SMD:R_0402_1005Metric, F.Cu at (131.4, 78.8)
- added R13: 130k, Resistor_SMD:R_0402_1005Metric, F.Cu at (134.3, 66.8)
- added R14: 10k, Resistor_SMD:R_0402_1005Metric, F.Cu at (134.3, 68.8)
- added R15: 1k, Resistor_SMD:R_0402_1005Metric, F.Cu at (134.3, 70.8)
- added R16: 22R, Resistor_SMD:R_0402_1005Metric, F.Cu at (134.3, 72.8)
- added R17: 22R, Resistor_SMD:R_0402_1005Metric, F.Cu at (134.3, 74.8)
- added R18: 22R, Resistor_SMD:R_0402_1005Metric, F.Cu at (134.3, 76.8)
- added R19: 22R, Resistor_SMD:R_0402_1005Metric, F.Cu at (134.3, 78.8)
- added R20: 22R, Resistor_SMD:R_0402_1005Metric, F.Cu at (137.3, 66.8)
- added R21: 22R, Resistor_SMD:R_0402_1005Metric, F.Cu at (137.3, 68.8)
- added R22: 4.7R, Resistor_SMD:R_0402_1005Metric, F.Cu at (137.3, 70.8)
- added R23: 4.7R, Resistor_SMD:R_0402_1005Metric, F.Cu at (137.3, 72.8)
- added R24: 4.7R, Resistor_SMD:R_0402_1005Metric, F.Cu at (137.3, 74.8)
- added R25: 130k, Resistor_SMD:R_0402_1005Metric, F.Cu at (131.4, 52.9)
- added R26: 10k, Resistor_SMD:R_0402_1005Metric, F.Cu at (131.4, 54.9)
- added R27: 1k, Resistor_SMD:R_0402_1005Metric, F.Cu at (131.4, 56.9)
- added R28: 130k, Resistor_SMD:R_0402_1005Metric, F.Cu at (131.4, 58.9)
- added R29: 10k, Resistor_SMD:R_0402_1005Metric, F.Cu at (131.4, 60.8)
- added R30: 1k, Resistor_SMD:R_0402_1005Metric, F.Cu at (131.4, 62.8)
- added R31: 130k, Resistor_SMD:R_0402_1005Metric, F.Cu at (134.3, 50.9)
- added R32: 10k, Resistor_SMD:R_0402_1005Metric, F.Cu at (134.3, 52.9)
- added R33: 1k, Resistor_SMD:R_0402_1005Metric, F.Cu at (134.3, 54.9)
- added R34: 22R, Resistor_SMD:R_0402_1005Metric, F.Cu at (134.3, 56.9)
- added R35: 22R, Resistor_SMD:R_0402_1005Metric, F.Cu at (134.3, 58.9)
- added R36: 22R, Resistor_SMD:R_0402_1005Metric, F.Cu at (134.3, 60.8)
- added R37: 22R, Resistor_SMD:R_0402_1005Metric, F.Cu at (134.3, 62.8)
- added R38: 22R, Resistor_SMD:R_0402_1005Metric, F.Cu at (137.3, 50.9)
- added R39: 22R, Resistor_SMD:R_0402_1005Metric, F.Cu at (137.3, 52.9)
- added R40: 4.7R, Resistor_SMD:R_0402_1005Metric, F.Cu at (137.3, 54.9)
- added R41: 4.7R, Resistor_SMD:R_0402_1005Metric, F.Cu at (137.3, 56.9)
- added R42: 4.7R, Resistor_SMD:R_0402_1005Metric, F.Cu at (137.3, 58.9)
- added R43: 130k, Resistor_SMD:R_0402_1005Metric, F.Cu at (114.1, 70.7)
- added R44: 10k, Resistor_SMD:R_0402_1005Metric, F.Cu at (114.1, 72.7)
- added R45: 1k, Resistor_SMD:R_0402_1005Metric, F.Cu at (114.1, 74.6)
- added R46: 130k, Resistor_SMD:R_0402_1005Metric, F.Cu at (114.1, 76.6)
- added R47: 10k, Resistor_SMD:R_0402_1005Metric, F.Cu at (114.1, 78.6)
- added R48: 1k, Resistor_SMD:R_0402_1005Metric, F.Cu at (114.1, 80.6)
- added R49: 130k, Resistor_SMD:R_0402_1005Metric, F.Cu at (117.0, 68.7)
- added R50: 10k, Resistor_SMD:R_0402_1005Metric, F.Cu at (117.0, 70.7)
- added R51: 1k, Resistor_SMD:R_0402_1005Metric, F.Cu at (117.0, 72.7)
- added R52: 22R, Resistor_SMD:R_0402_1005Metric, F.Cu at (117.0, 74.6)
- added R53: 22R, Resistor_SMD:R_0402_1005Metric, F.Cu at (117.0, 76.6)
- added R54: 22R, Resistor_SMD:R_0402_1005Metric, F.Cu at (117.0, 78.6)
- added R55: 22R, Resistor_SMD:R_0402_1005Metric, F.Cu at (117.0, 80.6)
- added R56: 22R, Resistor_SMD:R_0402_1005Metric, F.Cu at (119.9, 68.7)
- added R57: 22R, Resistor_SMD:R_0402_1005Metric, F.Cu at (119.9, 70.7)
- added R58: 4.7R, Resistor_SMD:R_0402_1005Metric, F.Cu at (119.9, 72.7)
- added R59: 4.7R, Resistor_SMD:R_0402_1005Metric, F.Cu at (119.9, 74.6)
- added R60: 4.7R, Resistor_SMD:R_0402_1005Metric, F.Cu at (119.9, 76.6)
- added R61: 130k, Resistor_SMD:R_0402_1005Metric, F.Cu at (131.4, 84.7)
- added R62: 10k, Resistor_SMD:R_0402_1005Metric, F.Cu at (116.9, 86.6)
- added R63: 10k, Resistor_SMD:R_0402_1005Metric, F.Cu at (131.4, 86.7)
- added R64: 1k, Resistor_SMD:R_0402_1005Metric, F.Cu at (131.4, 88.7)
- added R65: 130k, Resistor_SMD:R_0402_1005Metric, F.Cu at (131.4, 90.7)
- added R66: 10k, Resistor_SMD:R_0402_1005Metric, F.Cu at (131.4, 92.7)
- added R67: 1k, Resistor_SMD:R_0402_1005Metric, F.Cu at (131.4, 94.7)
- added R68: 130k, Resistor_SMD:R_0402_1005Metric, F.Cu at (134.3, 82.8)
- added R69: 10k, Resistor_SMD:R_0402_1005Metric, F.Cu at (134.3, 84.7)
- added R7: 130k, Resistor_SMD:R_0402_1005Metric, F.Cu at (131.4, 68.8)
- added R70: 1k, Resistor_SMD:R_0402_1005Metric, F.Cu at (134.3, 86.7)
- added R71: 22R, Resistor_SMD:R_0402_1005Metric, F.Cu at (134.3, 88.7)
- added R72: 22R, Resistor_SMD:R_0402_1005Metric, F.Cu at (134.3, 90.7)
- added R73: 22R, Resistor_SMD:R_0402_1005Metric, F.Cu at (134.3, 92.7)
- added R74: 22R, Resistor_SMD:R_0402_1005Metric, F.Cu at (134.3, 94.7)
- added R75: 22R, Resistor_SMD:R_0402_1005Metric, F.Cu at (137.3, 82.8)
- added R76: 22R, Resistor_SMD:R_0402_1005Metric, F.Cu at (137.3, 84.7)
- added R77: 4.7R, Resistor_SMD:R_0402_1005Metric, F.Cu at (137.3, 86.7)
- added R78: 4.7R, Resistor_SMD:R_0402_1005Metric, F.Cu at (137.3, 88.7)
- added R79: 4.7R, Resistor_SMD:R_0402_1005Metric, F.Cu at (137.3, 90.7)
- added R8: 10k, Resistor_SMD:R_0402_1005Metric, F.Cu at (131.4, 70.8)
- added R80: 10k, Resistor_SMD:R_0402_1005Metric, F.Cu at (150.8, 52.9)
- added R82: 10R, Resistor_SMD:R_0402_1005Metric, F.Cu at (124.9, 62.2)
- added R83: 100k, Resistor_SMD:R_0402_1005Metric, F.Cu at (124.7, 84.6)
- added R84: 8.66k, Resistor_SMD:R_0402_1005Metric, F.Cu at (124.7, 86.6)
- added R85: 10k, Resistor_SMD:R_0402_1005Metric, F.Cu at (150.8, 74.7)
- added R86: 10k, Resistor_SMD:R_0402_1005Metric, F.Cu at (150.8, 90.7)
- added R87: 10R, Resistor_SMD:R_0402_1005Metric, F.Cu at (124.9, 64.2)
- added R9: 1k, Resistor_SMD:R_0402_1005Metric, F.Cu at (131.4, 72.8)
- added U1: INA181A2IDBVR, easyeda_import:SOT-23-6_L2.9-W1.6-P0.95-LS2.8-BL, F.Cu at (125.9, 59.0)
- added U12: STM32G071GBU6, easyeda_import:UFQFPN-28_L4.0-W4.0-P0.50-BL, F.Cu at (152.1, 68.7)
- added U13: STM32G071GBU6, easyeda_import:UFQFPN-28_L4.0-W4.0-P0.50-BL, F.Cu at (152.1, 84.6)
- U4: value STM32G071GBU6 -> JSM6288Q; footprint easyeda_import:UFQFPN-28_L4.0-W4.0-P0.50-BL -> easyeda_import:VQFN-24_L4.0-W4.0-P0.50-TL-EP2.7
Connections:
- Q10 pad 5: GND_BAT -> GND
- Q10 pad 6: GND_BAT -> GND
- Q10 pad 7: GND_BAT -> GND
- Q10 pad 8: GND_BAT -> GND
- Q12 pad 5: GND_BAT -> GND
- Q12 pad 6: GND_BAT -> GND
- Q12 pad 7: GND_BAT -> GND
- Q12 pad 8: GND_BAT -> GND
- Q14 pad 5: GND_BAT -> GND
- Q14 pad 6: GND_BAT -> GND
- Q14 pad 7: GND_BAT -> GND
- Q14 pad 8: GND_BAT -> GND
- Q16 pad 5: GND_BAT -> GND
- Q16 pad 6: GND_BAT -> GND
- Q16 pad 7: GND_BAT -> GND
- Q16 pad 8: GND_BAT -> GND
- Q18 pad 5: GND_BAT -> GND
- Q18 pad 6: GND_BAT -> GND
- Q18 pad 7: GND_BAT -> GND
- Q18 pad 8: GND_BAT -> GND
- Q2 pad 5: GND_BAT -> GND
- Q2 pad 6: GND_BAT -> GND
- Q2 pad 7: GND_BAT -> GND
- Q2 pad 8: GND_BAT -> GND
- Q20 pad 5: GND_BAT -> GND
- Q20 pad 6: GND_BAT -> GND
- Q20 pad 7: GND_BAT -> GND
- Q20 pad 8: GND_BAT -> GND
- Q22 pad 5: GND_BAT -> GND
- Q22 pad 6: GND_BAT -> GND
- Q22 pad 7: GND_BAT -> GND
- Q22 pad 8: GND_BAT -> GND
- Q24 pad 5: GND_BAT -> GND
- Q24 pad 6: GND_BAT -> GND
- Q24 pad 7: GND_BAT -> GND
- Q24 pad 8: GND_BAT -> GND
- Q4 pad 5: GND_BAT -> GND
- Q4 pad 6: GND_BAT -> GND
- Q4 pad 7: GND_BAT -> GND
- Q4 pad 8: GND_BAT -> GND
- Q6 pad 5: GND_BAT -> GND
- Q6 pad 6: GND_BAT -> GND
- Q6 pad 7: GND_BAT -> GND
- Q6 pad 8: GND_BAT -> GND
- Q8 pad 5: GND_BAT -> GND
- Q8 pad 6: GND_BAT -> GND
- Q8 pad 7: GND_BAT -> GND
- Q8 pad 8: GND_BAT -> GND
- U10 pad 2: GND_BAT -> GND
- U2 pad 25: GND_BAT -> GND
- U3 pad 25: GND_BAT -> GND
- U4 pad 1: unconnected-(U4-PC14-OSC32_IN-Pad1) -> /BLDC DRIVE2/LIN1
- U4 pad 10: /STM32F051K8U7/BEMF.A -> Net-(U4-LO2)
- U4 pad 11: /STM32F051K8U7/BEMF.B -> Net-(U4-LO1)
- U4 pad 12: /STM32F051K8U7/BEMF.C -> /BLDC DRIVE2/C
- U4 pad 13: /STM32F051K8U7/LIN1 -> Net-(U4-HO3)
- U4 pad 14: /STM32F051K8U7/LIN2 -> /BLDC DRIVE2/BOOT3
- U4 pad 15: /STM32F051K8U7/LIN3 -> /BLDC DRIVE2/B
- U4 pad 16: /STM32F051K8U7/HIN1 -> Net-(U4-HO2)
- U4 pad 17: unconnected-(U4-PC6-Pad17) -> /BLDC DRIVE2/BOOT2
- U4 pad 18: /STM32F051K8U7/HIN2 -> /BLDC DRIVE2/A
- U4 pad 19: /STM32F051K8U7/HIN3 -> Net-(U4-HO1)
- U4 pad 2: unconnected-(U4-PC15-OSC32_OUT-Pad2) -> /BLDC DRIVE2/LIN2
- U4 pad 20: /STM32F051K8U7/SWDIO -> /BLDC DRIVE2/BOOT1
- U4 pad 21: /STM32F051K8U7/SWCLK -> unconnected-(U4-NC-Pad21)
- U4 pad 22: unconnected-(U4-PA15-Pad22) -> /BLDC DRIVE2/HIN1
- U4 pad 23: unconnected-(U4-PB3-Pad23) -> /BLDC DRIVE2/HIN2
- U4 pad 24: unconnected-(U4-PB4-Pad24) -> /BLDC DRIVE2/HIN3
- U4 pad 25: unconnected-(U4-PB5-Pad25) -> GND
- U4 pad 3: +3V3_FILT -> /BLDC DRIVE2/LIN3
- U4 pad 4: GND -> +10V_FILT
- U4 pad 5: /STM32F051K8U7/NRST -> unconnected-(U4-NC-Pad5)
- U4 pad 6: unconnected-(U4-PA0-Pad6) -> GND_BAT
- U4 pad 8: /STM32F051K8U7/DSHOT_RX -> unconnected-(U4-NC-Pad8)
- U4 pad 9: /STM32F051K8U7/BEMF.COMMON -> Net-(U4-LO3)
- U5 pad 1: /BLDC DRIVE2/LIN1 -> /BLDC DRIVE3/LIN1
- U5 pad 12: /BLDC DRIVE2/C -> /BLDC DRIVE3/C
- U5 pad 14: /BLDC DRIVE2/BOOT3 -> /BLDC DRIVE3/BOOT3
- U5 pad 15: /BLDC DRIVE2/B -> /BLDC DRIVE3/B
- U5 pad 17: /BLDC DRIVE2/BOOT2 -> /BLDC DRIVE3/BOOT2
- U5 pad 18: /BLDC DRIVE2/A -> /BLDC DRIVE3/A
- U5 pad 2: /BLDC DRIVE2/LIN2 -> /BLDC DRIVE3/LIN2
- U5 pad 20: /BLDC DRIVE2/BOOT1 -> /BLDC DRIVE3/BOOT1
- U5 pad 22: /BLDC DRIVE2/HIN1 -> /BLDC DRIVE3/HIN1
- U5 pad 23: /BLDC DRIVE2/HIN2 -> /BLDC DRIVE3/HIN2
- U5 pad 24: /BLDC DRIVE2/HIN3 -> /BLDC DRIVE3/HIN3
- U5 pad 25: GND_BAT -> GND
- U5 pad 3: /BLDC DRIVE2/LIN3 -> /BLDC DRIVE3/LIN3
- U6 pad 20: /STM32F051K8U6/SWDIO -> /SWDIO_M4
- U6 pad 21: /STM32F051K8U6/SWCLK -> /SWCLK_M4
- U6 pad 26: unconnected-(U6-PB6-Pad26) -> /STM32F051K8U6/KISS_TELEM
- U6 pad 27: unconnected-(U6-PB7-Pad27) -> /STM32F051K8U6/CURRENT_SENSE
- U6 pad 8: /STM32F051K8U6/DSHOT_RX -> /DSHOT_M4
- U7 pad 10: /STM32F051K8U8/BEMF.A -> /BLDC DRIVE2/BEMF.A
- U7 pad 11: /STM32F051K8U8/BEMF.B -> /BLDC DRIVE2/BEMF.B
- U7 pad 12: /STM32F051K8U8/BEMF.C -> /BLDC DRIVE2/BEMF.C
- U7 pad 13: /STM32F051K8U8/LIN1 -> /BLDC DRIVE2/LIN1
- U7 pad 14: /STM32F051K8U8/LIN2 -> /BLDC DRIVE2/LIN2
- U7 pad 15: /STM32F051K8U8/LIN3 -> /BLDC DRIVE2/LIN3
- U7 pad 16: /STM32F051K8U8/HIN1 -> /BLDC DRIVE2/HIN1
- U7 pad 18: /STM32F051K8U8/HIN2 -> /BLDC DRIVE2/HIN2
- U7 pad 19: /STM32F051K8U8/HIN3 -> /BLDC DRIVE2/HIN3
- U7 pad 20: /STM32F051K8U8/SWDIO -> /SWDIO_M1
- U7 pad 21: /STM32F051K8U8/SWCLK -> /SWCLK_M1
- U7 pad 26: unconnected-(U7-PB6-Pad26) -> /KISS_TELEM
- U7 pad 27: unconnected-(U7-PB7-Pad27) -> /CURRENT_SENSE
- U7 pad 8: /STM32F051K8U8/DSHOT_RX -> /DSHOT_M1
- U7 pad 9: /STM32F051K8U8/BEMF.COMMON -> /BLDC DRIVE2/BEMF.COMMON
