File: 4-in-1_ESC/DCDC.kicad_sch (KiCad schematic)
At the start: 11 parts, among them U10 LMR51610XDBVR, U11 AMS1117-3.3_C347222

Commit message: Schematic First Pass
Connections:
- net GND_BAT is gone; now on net GND: C74.2, C75.2, U10.2 (GND)
Other:
- note added: "10V BUCK"
- note added: "1A Synchronous Buck Converter with 4V to 65V Input Range"
- note added: "3V3 LDO"
- note added: "Arm Cortex-M0+ 32-bit MCU, up to 128 KB Flash, 36 KB RAM, 4x USART, timers, ADC, DAC, comm. I/Fs, 1.7-3.6V"
- note added: "TI LMR51610XDBVR"
- note added: "UMW AMS1117-3.3"
- moved on the sheet: C74, C75, C76, C77, C78, C79, L1, R83, R84, U10, U11
