File: 4-in-1_ESC/DCDC.kicad_sch (KiCad schematic)
At the start: 11 parts, among them U10 LMR51610XDBVR, U11 AMS1117-3.3_C347222

Commit message: update
Parts:
- C76, C77, C78, C79: footprint Capacitor_SMD:C_0402_1005Metric -> Capacitor_SMD:C_0201_0603Metric
- R83, R84: footprint Resistor_SMD:R_0402_1005Metric -> Resistor_SMD:R_0201_0603Metric
Changed lines of the file:
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@@
 			)
 		)
-		(property "Footprint" "Capacitor_SMD:C_0402_1005Metric"
+		(property "Footprint" "Capacitor_SMD:C_0201_0603Metric"
 			(at 132.08 107.95 0)
 			(hide yes)
@@
 			)
 		)
-		(property "Footprint" "Capacitor_SMD:C_0402_1005Metric"
+		(property "Footprint" "Capacitor_SMD:C_0201_0603Metric"
 			(at 102.87 99.06 0)
 			(hide yes)
@@
 			)
 		)
-		(property "Footprint" "Resistor_SMD:R_0402_1005Metric"
+		(property "Footprint" "Resistor_SMD:R_0201_0603Metric"
 			(at 116.84 111.76 0)
 			(hide yes)
@@
 			)
 		)
-		(property "Footprint" "Capacitor_SMD:C_0402_1005Metric"
+		(property "Footprint" "Capacitor_SMD:C_0201_0603Metric"
 			(at 193.04 106.68 0)
 			(hide yes)
@@
 			)
 		)
-		(property "Footprint" "Capacitor_SMD:C_0402_1005Metric"
+		(property "Footprint" "Capacitor_SMD:C_0201_0603Metric"
 			(at 247.65 109.22 0)
 			(hide yes)
@@
 			)
 		)
-		(property "Footprint" "Resistor_SMD:R_0402_1005Metric"
+		(property "Footprint" "Resistor_SMD:R_0201_0603Metric"
 			(at 116.84 105.41 0)
 			(hide yes)

Commit message: changes
Parts:
- removed U11: AMS1117-3.3_C347222, easyeda_import:SOT-223-4_L6.5-W3.5-P2.30-LS7.0-BR, symbol easyeda_import:AMS1117-3.3_C347222
- added U8: TLV76733DRVR, easyeda_import:WSON-6_L2.0-W2.0-P0.65-TL-EP, symbol easyeda_import:TLV76733DRVR
Connections:
- net +10V: now also U8.4 (EN), U8.6 (IN)
- net +3V3: now also U8.1 (OUT), U8.2 (FB/SNS)
- net GND: now also U8.3 (GND), U8.5 (GND), U8.7 (EP)
Other:
- note added: "1A, 16V positive voltage low dropout (LDO) linear regulator with adjustable and fixed output"
- note added: "TI TLV76733DRVR"
- note removed: "1A Synchronous Buck Converter with 4V to 65V Input Range"
- note removed: "UMW AMS1117-3.3"
- moved on the sheet: C78, C79

Commit message: Update
Parts:
- added C95: 100nF, Capacitor_SMD:C_0201_0603Metric, symbol Device:C_Small
- C77: value 2.2uF -> 22uF
- C78: value 10uF -> 1uF
- C79: value 22uF -> 2.2uF
- L1: value 4.7uH -> 56uH
Connections:
- net +10V: now also C95.1
- net GND: now also C95.2
Changed lines of the file:
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@@
 				(thickness 0.508)
 				(bold yes)
-				(color 255 255 255 1)
+				(color 255 0 0 1)
 			)
 			(justify left)
@@
 				(thickness 0.508)
 				(bold yes)
-				(color 255 255 255 1)
+				(color 255 0 0 1)
 			)
 			(justify left)
@@
 				(thickness 0.508)
 				(bold yes)
-				(color 255 255 255 1)
+				(color 255 0 0 1)
 			)
 			(justify left)
@@
 				(thickness 0.508)
 				(bold yes)
-				(color 255 255 255 1)
-			)
-			(justify left)
-		)
-	)
-	(text_box "VERF COMPONENTS"
-		(exclude_from_sim no)
-		(at 81.28 141.0494 0)
-		(size 33.02 10.0806)
-		(margins 0.9525 0.9525 0.9525 0.9525)
-		(stroke
-			(width 0)
-			(type solid)
-		)
-		(fill
-			(type color)
-			(color 255 229 191 1)
-		)
-		(effects
-			(font
-				(size 2.54 2.54)
-				(color 255 0 0 1)
-			)
-			(justify left top)
-		)
-	)
-	(text_box "ADD DIODE"
-		(exclude_from_sim no)
-		(at 81.28 134.62 0)
-		(size 33.02 5.9913)
-		(margins 0.9525 0.9525 0.9525 0.9525)
-		(stroke
-			(width 0)
-			(type solid)
-		)
-		(fill
-			(type color)
-			(color 255 229 191 1)
-		)
-		(effects
-			(font
-				(size 2.54 2.54)
 				(color 255 0 0 1)
 			)
-			(justify left top)
+			(justify left)
 		)
 	)
@@
 		)
 	)
-	(text_box "400kHz"
+	(text_box "L = (VIN_MAX − VOUT) / (IOUT × KIND) × VOUT / (VIN_MAX × fSW)\nL = 58.5 µH"
 		(exclude_from_sim no)
-		(at 107.95 90.17 0)
-		(size 12.7 3.9483)
+		(at 109.22 84.6724 0)
+		(size 46.99 8.0376)
 		(margins 0.9525 0.9525 0.9525 0.9525)
 		(stroke
@@
 		)
 	)
-	(text_box "ADD CAPS"
-		(exclude_from_sim no)
-		(at 204.47 133.35 0)
-		(size 33.02 5.9913)
-		(margins 0.9525 0.9525 0.9525 0.9525)
-		(stroke
-			(width 0)
-			(type solid)
-		)
-		(fill
-			(type color)
-			(color 255 229 191 1)
-		)
-		(effects
-			(font
-				(size 2.54 2.54)
-				(color 255 0 0 1)
-			)
-			(justify left top)
-		)
-	)
 	(junction
 		(at 209.55 110.49)
@@
 	)
 	(junction
+		(at 132.08 101.6)
+		(diameter 0)
+		(color 0 0 0 0)
+	)
+	(junction
 		(at 238.76 102.87)
 		(diameter 0)
@@
 	)
 	(junction
-		(at 62.23 99.06)
+		(at 142.24 101.6)
 		(diameter 0)
 		(color 0 0 0 0)
 	)
 	(junction
-		(at 78.74 99.06)
+		(at 62.23 99.06)
 		(diameter 0)
 		(color 0 0 0 0)
 	)
 	(junction
-		(at 44.45 99.06)
+		(at 78.74 99.06)
 		(diameter 0)
 		(color 0 0 0 0)
 	)
 	(junction
-		(at 132.08 101.6)
+		(at 44.45 99.06)
 		(diameter 0)
 		(color 0 0 0 0)
@@
 	(wire
 		(pts
+			(xy 142.24 101.6) (xy 142.24 105.41)
+		)
+		(stroke
+			(width 0)
+			(type default)
+		)
+	)
+	(wire
+		(pts
 			(xy 78.74 107.95) (xy 78.74 113.03)
 		)
@@
 	(wire
 		(pts
+			(xy 142.24 110.49) (xy 142.24 114.3)
+		)
+		(stroke
+			(width 0)
+			(type default)
+		)
+	)
+	(wire
+		(pts
 			(xy 195.58 113.03) (xy 209.55 113.03)
 		)
@@
 	(wire
 		(pts
-			(xy 132.08 100.33) (xy 132.08 101.6)
+			(xy 142.24 100.33) (xy 142.24 101.6)
 		)
 		(stroke
@@
 	(wire
 		(pts
+			(xy 142.24 101.6) (xy 132.08 101.6)
+		)
+		(stroke
+			(width 0)
+			(type default)
+		)
+	)
+	(wire
+		(pts
 			(xy 81.28 107.95) (xy 78.74 107.95)
 		)
@@
 	)
 	(symbol
+		(lib_id "Device:C_Small")
+		(at 142.24 107.95 0)
+		(unit 1)
+		(body_style 1)
+		(exclude_from_sim no)
+		(in_bom yes)
+		(on_board yes)
+		(in_pos_files yes)
+		(dnp no)
+		(fields_autoplaced yes)
+		(property "Reference" "C95"
+			(at 144.78 106.6862 0)
+			(show_name no)
+			(do_not_autoplace no)
+			(effects
+				(font
+					(size 1.27 1.27)
+				)
+				(justify left)
+			)
+		)
+		(property "Value" "100nF"
+			(at 144.78 109.2262 0)
+			(show_name no)
+			(do_not_autoplace no)
+			(effects
+				(font
+					(size 1.27 1.27)
+				)
+				(justify left)
+			)
+		)
+		(property "Footprint" "Capacitor_SMD:C_0201_0603Metric"
+			(at 142.24 107.95 0)
+			(hide yes)
+			(show_name no)
+			(do_not_autoplace no)
+			(effects
+				(font
+					(size 1.27 1.27)
+				)
+			)
+		)
+		(property "Datasheet" ""
+			(at 142.24 107.95 0)
+			(hide yes)
+			(show_name no)
+			(do_not_autoplace no)
+			(effects
+				(font
+					(size 1.27 1.27)
+				)
+			)
+		)
+		(property "Description" "Unpolarized capacitor, small symbol"
+			(at 142.24 107.95 0)
+			(hide yes)
+			(show_name no)
+			(do_not_autoplace no)
+			(effects
+				(font
+					(size 1.27 1.27)
+				)
+			)
+		)
+		(pin "1"
+		)
+		(pin "2"
+		)
+		(instances
+			(project "4-in-1_ESC"
+				(path "/885456b2-b92d-459f-a061-5f970a420f96/d2328bdd-1cef-4230-98f7-ffdd8d70ee2d"
+					(reference "C95")
+					(unit 1)
+				)
+			)
+		)
+	)
+	(symbol
 		(lib_id "power:GND")
 		(at 132.08 114.3 0)
@@
 			)
 		)
-		(property "Value" "2.2uF"
+		(property "Value" "22uF"
 			(at 134.62 109.2135 0)
 			(show_name no)
@@
 	(symbol
 		(lib_id "power:GND")
+		(at 142.24 114.3 0)
+		(unit 1)
+		(body_style 1)
+		(exclude_from_sim no)
+		(in_bom yes)
+		(on_board yes)
+		(in_pos_files yes)
+		(dnp no)
+		(fields_autoplaced yes)
+		(property "Reference" "#PWR092"
+			(at 142.24 120.65 0)
+			(hide yes)
+			(show_name no)
+			(do_not_autoplace no)
+			(effects
+				(font
+					(size 1.27 1.27)
+				)
+			)
+		)
+		(property "Value" "GND"
+			(at 142.24 119.38 0)
+			(show_name no)
+			(do_not_autoplace no)
+			(effects
+				(font
+					(size 1.27 1.27)
+				)
+			)
+		)
+		(property "Footprint" ""
+			(at 142.24 114.3 0)
+			(hide yes)
+			(show_name no)
+			(do_not_autoplace no)
+			(effects
+				(font
+					(size 1.27 1.27)
+				)
+			)
+		)
+		(property "Datasheet" ""
+			(at 142.24 114.3 0)
+			(hide yes)
+			(show_name no)
+			(do_not_autoplace no)
+			(effects
+				(font
+					(size 1.27 1.27)
+				)
+			)
+		)
+		(property "Description" "Power symbol creates a global label with name \"GND\" , ground"
+			(at 142.24 114.3 0)
+			(hide yes)
+			(show_name no)
+			(do_not_autoplace no)
+			(effects
+				(font
+					(size 1.27 1.27)
+				)
+			)
+		)
+		(pin "1"
+		)
+		(instances
+			(project "4-in-1_ESC"
+				(path "/885456b2-b92d-459f-a061-5f970a420f96/d2328bdd-1cef-4230-98f7-ffdd8d70ee2d"
+					(reference "#PWR092")
+					(unit 1)
+				)
+			)
+		)
+	)
+	(symbol
+		(lib_id "power:GND")
 		(at 116.84 114.3 0)
 		(unit 1)
@@
 			)
 		)
-		(property "Value" "10uF"
+		(property "Value" "1uF"
 			(at 198.12 109.2262 0)
 			(show_name no)
@@
 	(symbol
 		(lib_id "power:+10V")
-		(at 132.08 100.33 0)
+		(at 142.24 100.33 0)
 		(unit 1)
 		(body_style 1)
@@
 		(fields_autoplaced yes)
 		(property "Reference" "#PWR085"
-			(at 132.08 104.14 0)
+			(at 142.24 104.14 0)
 			(hide yes)
 			(show_name no)
@@
 		)
 		(property "Value" "+10V"
-			(at 132.08 95.25 0)
+			(at 142.24 95.25 0)
 			(show_name no)
 			(do_not_autoplace no)
@@
 		)
 		(property "Footprint" ""
-			(at 132.08 100.33 0)
+			(at 142.24 100.33 0)
 			(hide yes)
 			(show_name no)
@@
 		)
 		(property "Datasheet" ""
-			(at 132.08 100.33 0)
+			(at 142.24 100.33 0)
 			(hide yes)
 			(show_name no)
@@
 		)
 		(property "Description" "Power symbol creates a global label with name \"+10V\""
-			(at 132.08 100.33 0)
+			(at 142.24 100.33 0)
 			(hide yes)
 			(show_name no)
@@
 			)
 		)
-		(property "Value" "22uF"
+		(property "Value" "2.2uF"
 			(at 250.19 109.2262 0)
 			(show_name no)
@@
 			)
 		)
-		(property "Value" "4.7uH"
+		(property "Value" "56uH"
 			(at 113.03 99.06 90)
 			(show_name no)
