File: 4-in-1_ESC/BLDCDrive.kicad_sch (KiCad schematic)
At the start: 39 parts, among them Q1 BSC070N10NS3G, Q2 BSC070N10NS3G, Q3 BSC070N10NS3G, Q4 BSC070N10NS3G, Q5 BSC070N10NS3G, Q6 BSC070N10NS3G, U2 JSM6288Q

Commit message: update
Parts:
- C26, C27, C28: value 10nF -> 1nF; footprint Capacitor_SMD:C_0402_1005Metric -> Capacitor_SMD:C_0201_0603Metric
- C29, C30, C31, C32, C33, C54, C67: footprint Capacitor_SMD:C_0402_1005Metric -> Capacitor_SMD:C_0201_0603Metric
- R11, R14, R16, R17, R18, R19, R20, R21, R22, R23, R24, R45, R49, R67, R8, R82, R90, R96: footprint Resistor_SMD:R_0402_1005Metric -> Resistor_SMD:R_0201_0603Metric
Connections:
- net GND_BAT is gone; now on net GND: U2.6 (COM)

Commit message: changes
Changed lines of the file:
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@@
+		)
+	)
+	(text_box "SMALLER DIODES"
+		(exclude_from_sim no)
+		(at 260.35 140.97 0)
+		(size 33.02 10.0806)
+		(margins 0.9525 0.9525 0.9525 0.9525)
+		(stroke
+			(width 0)
+			(type solid)
+		)
+		(fill
+			(type color)
+			(color 255 229 191 1)
+		)
+		(effects
+			(font
+				(size 2.54 2.54)
+				(color 255 0 0 1)
+			)
+			(justify left top)
 		)
 	)

Commit message: Schematic Updates
Parts:
- removed C31: 4.7uF, Capacitor_SMD:C_0201_0603Metric, symbol Device:C_Small
- removed R24: 2.2R, Resistor_SMD:R_0201_0603Metric, symbol Device:R_Small_US
- added C46: 4.7uF 25V X5R, Capacitor_SMD:C_01005_0402Metric, symbol Device:C_Small
- added R28: 4.7R, Resistor_SMD:R_0201_0603Metric, symbol Device:R_Small_US
- C29, C30: value 4.7uF -> 4.7uF 25V X5R; footprint Capacitor_SMD:C_0201_0603Metric -> Capacitor_SMD:C_01005_0402Metric; LCSC_Part_Number (none) -> C2858031
- D1, D2, D3: value DSF1D E1D -> CDSQC4148-HF; footprint Diode_SMD:D_SOD-123F -> Diode_SMD:D_0402_1005Metric; LCSC_Part_Number C5365387 -> C6341459
- R22, R23: value 2.2R -> 4.7R; LCSC_Part_Number (none) -> C474426
Connections:
- net +10V: now also R28.2
- net BOOT3: now also C46.1
- net C: now also C46.2
- net at D3.2 (A): now also R28.1
Other:
- moved on the sheet: C29, D1, R22
