File: 4-in-1_ESC/BLDCDrive.kicad_sch (KiCad schematic)
At the start: 39 parts, among them Q1 BSC070N10NS3G, Q2 BSC070N10NS3G, Q3 BSC070N10NS3G, Q4 BSC070N10NS3G, Q5 BSC070N10NS3G, Q6 BSC070N10NS3G, U2 JSM6288Q

Commit message: Update
Parts:
- removed C53, C99: 4.7uF 25V X5R, Capacitor_SMD:C_0402_1005Metric, symbol Device:C_Small
- added C29, C30: 4.7uF 25V X5R, Capacitor_SMD:C_01005_0402Metric, symbol Device:C_Small
- C46: footprint Capacitor_SMD:C_0402_1005Metric -> Capacitor_SMD:C_01005_0402Metric
Connections:
- net A: now also C29.2
- net B: now also C30.2
- net BOOT1: now also C29.1
- net BOOT2: now also C30.1
Changed lines of the file:
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@@
 				(thickness 0.508)
 				(bold yes)
-				(color 255 0 0 1)
+				(color 255 255 255 1)
 			)
 			(justify left)
@@
 				(thickness 0.508)
 				(bold yes)
-				(color 255 0 0 1)
+				(color 255 255 255 1)
 			)
 			(justify left)
@@
 				(thickness 0.508)
 				(bold yes)
-				(color 255 0 0 1)
+				(color 255 255 255 1)
 			)
 			(justify left)
@@
 	)
 	(symbol
-		(lib_id "Device:C_Small")
-		(at 208.28 69.85 0)
-		(unit 1)
-		(body_style 1)
-		(exclude_from_sim no)
-		(in_bom yes)
-		(on_board yes)
-		(in_pos_files yes)
-		(dnp no)
-		(fields_autoplaced yes)
-		(property "Reference" "C99"
-			(at 210.82 68.5862 0)
-			(show_name no)
-			(do_not_autoplace no)
-			(effects
-				(font
-					(size 1.27 1.27)
-				)
-				(justify left)
-			)
-		)
-		(property "Value" "4.7uF 25V X5R"
-			(at 210.82 71.1262 0)
-			(show_name no)
-			(do_not_autoplace no)
-			(effects
-				(font
-					(size 1.27 1.27)
-				)
-				(justify left)
-			)
-		)
-		(property "Footprint" "Capacitor_SMD:C_0402_1005Metric"
-			(at 208.28 69.85 0)
-			(hide yes)
-			(show_name no)
-			(do_not_autoplace no)
-			(effects
-				(font
-					(size 1.27 1.27)
-				)
-			)
-		)
-		(property "Datasheet" ""
-			(at 208.28 69.85 0)
-			(hide yes)
-			(show_name no)
-			(do_not_autoplace no)
-			(effects
-				(font
-					(size 1.27 1.27)
-				)
-			)
-		)
-		(property "Description" "Unpolarized capacitor, small symbol"
-			(at 208.28 69.85 0)
-			(hide yes)
-			(show_name no)
-			(do_not_autoplace no)
-			(effects
-				(font
-					(size 1.27 1.27)
-				)
-			)
-		)
-		(property "LCSC_Part_Number" "C2858031"
-			(at 208.28 69.85 0)
-			(hide yes)
-			(show_name no)
-			(do_not_autoplace no)
-			(effects
-				(font
-					(size 1.27 1.27)
-				)
-			)
-		)
-		(pin "2"
-		)
-		(pin "1"
-		)
-		(instances
-			(project "4-in-1_ESC"
-				(path "/885456b2-b92d-459f-a061-5f970a420f96/24433638-03b1-4fac-9fb8-4bfe6ef19744"
-					(reference "C101")
-					(unit 1)
-				)
-				(path "/885456b2-b92d-459f-a061-5f970a420f96/77df452c-e4f2-43e0-967b-d0520b07b85a"
-					(reference "C100")
-					(unit 1)
-				)
-				(path "/885456b2-b92d-459f-a061-5f970a420f96/b59eefb5-17fe-40a6-bf35-994f052afcc0"
-					(reference "C99")
-					(unit 1)
-				)
-				(path "/885456b2-b92d-459f-a061-5f970a420f96/e58120a8-7607-4f33-8e63-95006a082acf"
-					(reference "C102")
-					(unit 1)
-				)
-			)
-		)
-	)
-	(symbol
 		(lib_id "Device:R_Small_US")
 		(at 76.2 106.68 180)
@@
 	)
 	(symbol
+		(lib_id "Device:C_Small")
+		(at 208.28 86.36 0)
+		(unit 1)
+		(body_style 1)
+		(exclude_from_sim no)
+		(in_bom yes)
+		(on_board yes)
+		(in_pos_files yes)
+		(dnp no)
+		(fields_autoplaced yes)
+		(property "Reference" "C30"
+			(at 210.82 85.0962 0)
+			(show_name no)
+			(do_not_autoplace no)
+			(effects
+				(font
+					(size 1.27 1.27)
+				)
+				(justify left)
+			)
+		)
+		(property "Value" "4.7uF 25V X5R"
+			(at 210.82 87.6362 0)
+			(show_name no)
+			(do_not_autoplace no)
+			(effects
+				(font
+					(size 1.27 1.27)
+				)
+				(justify left)
+			)
+		)
+		(property "Footprint" "Capacitor_SMD:C_01005_0402Metric"
+			(at 208.28 86.36 0)
+			(hide yes)
+			(show_name no)
+			(do_not_autoplace no)
+			(effects
+				(font
+					(size 1.27 1.27)
+				)
+			)
+		)
+		(property "Datasheet" ""
+			(at 208.28 86.36 0)
+			(hide yes)
+			(show_name no)
+			(do_not_autoplace no)
+			(effects
+				(font
+					(size 1.27 1.27)
+				)
+			)
+		)
+		(property "Description" "Unpolarized capacitor, small symbol"
+			(at 208.28 86.36 0)
+			(hide yes)
+			(show_name no)
+			(do_not_autoplace no)
+			(effects
+				(font
+					(size 1.27 1.27)
+				)
+			)
+		)
+		(property "LCSC_Part_Number" "C2858031"
+			(at 208.28 86.36 0)
+			(hide yes)
+			(show_name no)
+			(do_not_autoplace no)
+			(effects
+				(font
+					(size 1.27 1.27)
+				)
+			)
+		)
+		(pin "2"
+		)
+		(pin "1"
+		)
+		(instances
+			(project "4-in-1_ESC"
+				(path "/885456b2-b92d-459f-a061-5f970a420f96/24433638-03b1-4fac-9fb8-4bfe6ef19744"
+					(reference "C38")
+					(unit 1)
+				)
+				(path "/885456b2-b92d-459f-a061-5f970a420f96/77df452c-e4f2-43e0-967b-d0520b07b85a"
+					(reference "C31")
+					(unit 1)
+				)
+				(path "/885456b2-b92d-459f-a061-5f970a420f96/b59eefb5-17fe-40a6-bf35-994f052afcc0"
+					(reference "C30")
+					(unit 1)
+				)
+				(path "/885456b2-b92d-459f-a061-5f970a420f96/e58120a8-7607-4f33-8e63-95006a082acf"
+					(reference "C39")
+					(unit 1)
+				)
+			)
+		)
+	)
+	(symbol
 		(lib_id "Device:R_Small_US")
 		(at 180.34 50.8 90)
@@
 			)
 		)
-		(property "Footprint" "Capacitor_SMD:C_0402_1005Metric"
+		(property "Footprint" "Capacitor_SMD:C_01005_0402Metric"
 			(at 208.28 102.87 0)
 			(hide yes)
@@
 	)
 	(symbol
-		(lib_id "Device:C_Small")
-		(at 208.28 86.36 0)
-		(unit 1)
-		(body_style 1)
-		(exclude_from_sim no)
-		(in_bom yes)
-		(on_board yes)
-		(in_pos_files yes)
-		(dnp no)
-		(fields_autoplaced yes)
-		(property "Reference" "C53"
-			(at 210.82 85.0962 0)
-			(show_name no)
-			(do_not_autoplace no)
-			(effects
-				(font
-					(size 1.27 1.27)
-				)
-				(justify left)
-			)
-		)
-		(property "Value" "4.7uF 25V X5R"
-			(at 210.82 87.6362 0)
-			(show_name no)
-			(do_not_autoplace no)
-			(effects
-				(font
-					(size 1.27 1.27)
-				)
-				(justify left)
-			)
-		)
-		(property "Footprint" "Capacitor_SMD:C_0402_1005Metric"
-			(at 208.28 86.36 0)
-			(hide yes)
-			(show_name no)
-			(do_not_autoplace no)
-			(effects
-				(font
-					(size 1.27 1.27)
-				)
-			)
-		)
-		(property "Datasheet" ""
-			(at 208.28 86.36 0)
-			(hide yes)
-			(show_name no)
-			(do_not_autoplace no)
-			(effects
-				(font
-					(size 1.27 1.27)
-				)
-			)
-		)
-		(property "Description" "Unpolarized capacitor, small symbol"
-			(at 208.28 86.36 0)
-			(hide yes)
-			(show_name no)
-			(do_not_autoplace no)
-			(effects
-				(font
-					(size 1.27 1.27)
-				)
-			)
-		)
-		(property "LCSC_Part_Number" "C2858031"
-			(at 208.28 86.36 0)
-			(hide yes)
-			(show_name no)
-			(do_not_autoplace no)
-			(effects
-				(font
-					(size 1.27 1.27)
-				)
-			)
-		)
-		(pin "2"
-		)
-		(pin "1"
-		)
-		(instances
-			(project "4-in-1_ESC"
-				(path "/885456b2-b92d-459f-a061-5f970a420f96/24433638-03b1-4fac-9fb8-4bfe6ef19744"
-					(reference "C97")
-					(unit 1)
-				)
-				(path "/885456b2-b92d-459f-a061-5f970a420f96/77df452c-e4f2-43e0-967b-d0520b07b85a"
-					(reference "C96")
-					(unit 1)
-				)
-				(path "/885456b2-b92d-459f-a061-5f970a420f96/b59eefb5-17fe-40a6-bf35-994f052afcc0"
-					(reference "C53")
-					(unit 1)
-				)
-				(path "/885456b2-b92d-459f-a061-5f970a420f96/e58120a8-7607-4f33-8e63-95006a082acf"
-					(reference "C98")
-					(unit 1)
-				)
-			)
-		)
-	)
-	(symbol
 		(lib_id "power:VBUS")
 		(at 167.64 77.47 0)
@@
 					(unit 1)
 				)
+			)
+		)
+	)
+	(symbol
+		(lib_id "Device:C_Small")
+		(at 208.28 69.85 0)
+		(unit 1)
+		(body_style 1)
+		(exclude_from_sim no)
+		(in_bom yes)
+		(on_board yes)
+		(in_pos_files yes)
+		(dnp no)
+		(fields_autoplaced yes)
+		(property "Reference" "C29"
+			(at 210.82 68.5862 0)
+			(show_name no)
+			(do_not_autoplace no)
+			(effects
+				(font
+					(size 1.27 1.27)
+				)
+				(justify left)
+			)
+		)
+		(property "Value" "4.7uF 25V X5R"
+			(at 210.82 71.1262 0)
+			(show_name no)
+			(do_not_autoplace no)
+			(effects
+				(font
+					(size 1.27 1.27)
+				)
+				(justify left)
+			)
+		)
+		(property "Footprint" "Capacitor_SMD:C_01005_0402Metric"
+			(at 208.28 69.85 0)
+			(hide yes)
+			(show_name no)
+			(do_not_autoplace no)
+			(effects
+				(font
+					(size 1.27 1.27)
+				)
+			)
+		)
+		(property "Datasheet" ""
+			(at 208.28 69.85 0)
+			(hide yes)
+			(show_name no)
+			(do_not_autoplace no)
+			(effects
+				(font
+					(size 1.27 1.27)
+				)
+			)
+		)
+		(property "Description" "Unpolarized capacitor, small symbol"
+			(at 208.28 69.85 0)
+			(hide yes)
+			(show_name no)
+			(do_not_autoplace no)
+			(effects
+				(font
+					(size 1.27 1.27)
+				)
+			)
+		)
+		(property "LCSC_Part_Number" "C2858031"
+			(at 208.28 69.85 0)
+			(hide yes)
+			(show_name no)
+			(do_not_autoplace no)
+			(effects
+				(font
+					(size 1.27 1.27)
+				)
+			)
+		)
+		(pin "2"
+		)
+		(pin "1"
+		)
+		(instances
+			(project "4-in-1_ESC"
+				(path "/885456b2-b92d-459f-a061-5f970a420f96/24433638-03b1-4fac-9fb8-4bfe6ef19744"
+					(reference "C45")
+					(unit 1)
+				)
+				(path "/885456b2-b92d-459f-a061-5f970a420f96/77df452c-e4f2-43e0-967b-d0520b07b85a"
+					(reference "C37")
+					(unit 1)
+				)
+				(path "/885456b2-b92d-459f-a061-5f970a420f96/b59eefb5-17fe-40a6-bf35-994f052afcc0"
+					(reference "C29")
+					(unit 1)
+				)
+				(path "/885456b2-b92d-459f-a061-5f970a420f96/e58120a8-7607-4f33-8e63-95006a082acf"
+					(reference "C53")
+					(unit 1)
+				)
