File: 4-in-1_ESC/4-in-1_ESC.kicad_sch (KiCad schematic)
At the start: 41 parts, among them CN2 SM07B-SRSS-TB, J1 BLDC Solder Pads, J2 BLDC Solder Pads, J3 BLDC Solder Pads, J4 BLDC Solder Pads, U1 INA180A2IDBVR

Commit message: Update
Parts:
- removed C103, C104: 10uF, Capacitor_SMD:C_1210_3225Metric, symbol Device:C_Small
- removed R1, R2: 0.5 6W, easyeda_import:RES-SMD_L6.3-W3.2_R2512, symbol easyeda_import:ASR-M-3-0.5F
- added CN1: SM10B-SRSS-TB, easyeda_import:CONN-SMD_10P-P1.00_SM10B-SRSS-TB-LF-SN, symbol easyeda_import:SM10B-SRSS-TB
- added R1: 0.2m 6W SHUNT, easyeda_import:RES-SMD_L6.3-W3.1-1, symbol easyeda_import:ASR-M-3-0.25F
- NT1: footprint NetTie:NetTie-2_SMD_Pad0.5mm -> NetTie:NetTie-2_SMD_Pad2.0mm
Connections:
- net +3V3: now also CN1.1
- net GND: now also CN1.10, CN1.11, CN1.12, R1.1
- net SWCLK_M1: now also CN1.3
- net SWCLK_M2: now also CN1.5
- net SWCLK_M3: now also CN1.7
- net SWCLK_M4: now also CN1.9
- net SWDIO_M1: now also CN1.2
- net SWDIO_M2: now also CN1.4
- net SWDIO_M3: now also CN1.6
- net SWDIO_M4: now also CN1.8
- net at J5.2 (-), U1.4 (IN-): now also R1.2
Other:
- note added: "JST-SH 10 PIN -> DEBUG"
- moved on the sheet: CN2, NT1, R116, R117, R118, R119, R120, R121
