File: 4-in-1_ESC/STM_MCU.kicad_sch (KiCad schematic)
At the start: 15 parts, among them U12 STM32G071GBU6

Commit message: Update
Parts:
- removed TP1, TP13, TP5, TP9: TestPoint, TestPoint:TestPoint_Pad_D1.0mm, symbol Connector:TestPoint
Other:
- note removed: "PROGRAMMING TEST POINTS"
