File: 4-in-1_ESC.kicad_sch (KiCad schematic)
At the start: 39 parts, among them CN1 SM10B-SRSS-TB, CN2 SM07B-SRSS-TB, J1 BLDC Solder Pads, J2 BLDC Solder Pads, J3 BLDC Solder Pads, J4 BLDC Solder Pads, U1 INA180A2IDBVR

Commit message: update
Parts:
- removed R1: 0.2m 6W SHUNT, easyeda_import:RES-SMD_L6.3-W3.1-1, symbol easyeda_import:ASR-M-3-0.25F
- added R1, R2: 0.5 6W, easyeda_import:RES-SMD_L6.3-W3.2_R2512, symbol easyeda_import:ASR-M-3-0.5F
Connections:
- net GND: now also R1.2, R2.2
- net at J5.2 (-), U1.4 (IN-): now also R1.1, R2.1
Other:
- moved on the sheet: NT1
