File: 4-in-1_ESC.kicad_pcb (KiCad board)
At the start: 6 copper layers, 42.7 x 40.2 mm, 246 parts, among them CN1 SM10B-SRSS-TB, CN2 SM07B-SRSS-TB, J1 BLDC Solder Pads, J2 BLDC Solder Pads, J3 BLDC Solder Pads, J4 BLDC Solder Pads, Q1 BSC070N10NS3G, Q10 BSC070N10NS3G, Q11 BSC070N10NS3G, Q12 BSC070N10NS3G, Q13 BSC070N10NS3G, Q14 BSC070N10NS3G, Q15 BSC070N10NS3G, Q16 BSC070N10NS3G, Q17 BSC070N10NS3G, Q18 BSC070N10NS3G, Q19 BSC070N10NS3G, Q2 BSC070N10NS3G, Q20 BSC070N10NS3G, Q21 BSC070N10NS3G, Q22 BSC070N10NS3G, Q23 BSC070N10NS3G, Q24 BSC070N10NS3G, Q3 BSC070N10NS3G, Q4 BSC070N10NS3G, Q5 BSC070N10NS3G, Q6 BSC070N10NS3G, Q7 BSC070N10NS3G, Q8 BSC070N10NS3G, Q9 BSC070N10NS3G, U1 INA180A2IDBVR, U10 LMR51610XDBVR, U12 STM32G071GBU6, U13 STM32G071GBU6, U2 JSM6288Q, U3 JSM6288Q, U4 JSM6288Q, U5 JSM6288Q, U6 STM32G071GBU6, U7 STM32G071GBU6, U8 TLV76733DRVR

Commit message: update
Parts:
- added C95: 100nF, Capacitor_SMD:C_0201_0603Metric, B.Cu at (149.3, 92.5)
- added R2: 0.5 6W, easyeda_import:RES-SMD_L6.3-W3.2_R2512, B.Cu at (147.9, 84.7)
- C77: value 2.2uF -> 22uF
- C78: value 10uF -> 1uF
- C79: value 22uF -> 2.2uF
- R1: value 0.2m 6W SHUNT -> 0.5 6W; footprint easyeda_import:RES-SMD_L6.3-W3.1-1 -> easyeda_import:RES-SMD_L6.3-W3.2_R2512
- moved C16 63.3 mm to (144.3, 102.5)
- moved C23 54.1 mm to (144.3, 96.1)
- moved C22 52.9 mm to (150.3, 102.5), turned to 180 degrees
- moved C21 50.8 mm to (144.3, 92.9)
- moved C20 50.1 mm to (144.3, 89.7)
- moved C93 49.7 mm to (150.3, 99.4), turned to 180 degrees
- moved C19 49.5 mm to (144.3, 86.5)
- moved C92 49.2 mm to (150.3, 96.1), turned to 180 degrees
- moved C66 48.5 mm to (150.3, 93.0), turned to 180 degrees
- moved C25 48.0 mm to (150.3, 89.8), turned to 180 degrees
- moved C94 47.8 mm to (144.3, 99.3)
- moved NT1 17.6 mm to (116.3, 93.3)
- moved U1 5.86 mm to (151.1, 84.5), turned to 180 degrees
- moved R1 3.80 mm to (143.9, 84.7), turned to -90 degrees
- moved Q4 1.00 mm to (133.0, 88.9)
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Connections:
- R1 pad 1: GND -> Net-(J5--)
- R1 pad 2: Net-(J5--) -> GND

Commit message: Update
Parts:
- removed C29, C30, C31, C37, C38, C39, C45: 4.7uF 25V X5R, Capacitor_SMD:C_01005_0402Metric
- removed CN1: SM10B-SRSS-TB, easyeda_import:CONN-SMD_10P-P1.00_SM10B-SRSS-TB-LF-SN
- added C100: 4.7uF 25V X5R, Capacitor_SMD:C_0402_1005Metric, B.Cu at (140.6, 107.2)
- added C101: 4.7uF 25V X5R, Capacitor_SMD:C_0402_1005Metric, B.Cu at (151.1, 94.4)
- added C102: 4.7uF 25V X5R, Capacitor_SMD:C_0402_1005Metric, B.Cu at (151.1, 107.1)
- added C103: 10uF, Capacitor_SMD:C_1210_3225Metric, F.Cu at (150.1, 89.8)
- added C104: 10uF, Capacitor_SMD:C_1210_3225Metric, F.Cu at (144.4, 89.8)
- added C96: 4.7uF 25V X5R, Capacitor_SMD:C_0402_1005Metric, B.Cu at (143.2, 109.8)
- added C97: 4.7uF 25V X5R, Capacitor_SMD:C_0402_1005Metric, B.Cu at (154.3, 96.9)
- added C98: 4.7uF 25V X5R, Capacitor_SMD:C_0402_1005Metric, B.Cu at (153.6, 109.6)
- added C99: 4.7uF 25V X5R, Capacitor_SMD:C_0402_1005Metric, B.Cu at (141.2, 94.2)
- added TP1: TestPoint, TestPoint:TestPoint_Pad_D1.0mm, B.Cu at (94.6, 86.8)
- added TP10: TestPoint, TestPoint:TestPoint_Pad_D1.0mm, B.Cu at (99.6, 92.9)
- added TP11: TestPoint, TestPoint:TestPoint_Pad_D1.0mm, B.Cu at (104.7, 92.9)
- added TP12: TestPoint, TestPoint:TestPoint_Pad_D1.0mm, B.Cu at (109.7, 92.9)
- added TP13: TestPoint, TestPoint:TestPoint_Pad_D1.0mm, B.Cu at (94.6, 96.0)
- added TP14: TestPoint, TestPoint:TestPoint_Pad_D1.0mm, B.Cu at (99.6, 96.0)
- added TP15: TestPoint, TestPoint:TestPoint_Pad_D1.0mm, B.Cu at (104.7, 96.0)
- added TP16: TestPoint, TestPoint:TestPoint_Pad_D1.0mm, B.Cu at (109.7, 96.0)
- added TP2: TestPoint, TestPoint:TestPoint_Pad_D1.0mm, B.Cu at (99.6, 86.8)
- added TP3: TestPoint, TestPoint:TestPoint_Pad_D1.0mm, B.Cu at (104.7, 86.8)
- added TP4: TestPoint, TestPoint:TestPoint_Pad_D1.0mm, B.Cu at (109.7, 86.8)
- added TP5: TestPoint, TestPoint:TestPoint_Pad_D1.0mm, B.Cu at (94.6, 89.9)
- added TP6: TestPoint, TestPoint:TestPoint_Pad_D1.0mm, B.Cu at (99.6, 89.9)
- added TP7: TestPoint, TestPoint:TestPoint_Pad_D1.0mm, B.Cu at (104.7, 89.9)
- added TP8: TestPoint, TestPoint:TestPoint_Pad_D1.0mm, B.Cu at (109.7, 89.9)
- added TP9: TestPoint, TestPoint:TestPoint_Pad_D1.0mm, B.Cu at (94.6, 92.9)
- C26, C27, C28, C32, C33, C34, C35, C36, C40, C41, C42, C43, C44, C48, C49, C50, C51, C52, C54, C55, C56, C57, C60, C61, C62, C63, C64, C65, C67, C68, C69, C70, C71, C72, C73, C80, C81, C83, C84, C85, C87, C88, C89, C90, CN2, D1, D10, D11, D12, D13, D14, D15, D16, D2, D3, D4, D5, D6, D7, D8, D9, FB10, FB11, FB12, FB5, FB6, FB7, FB8, FB9, R100, R101, R102, R103, R104, R105, R106, R107, R11, R116, R117, R118, R119, R14, R16, R17, R18, R19, R20, R21, R22, R26, R27, R28, R29, R30, R31, R32, R33, R34, R35, R36, R37, R38, R39, R40, R44, R45, R47, R48, R49, R50, R51, R52, R53, R54, R55, R56, R57, R58, R61, R62, R63, R64, R65, R66, R67, R68, R69, R70, R71, R72, R73, R74, R75, R76, R77, R8, R80, R82, R85, R86, R87, R88, R89, R90, R91, R92, R93, R94, R95, R96, R97, R98, R99, TH1, TH2, TH3, TH4, U12, U13, U2, U3, U4, U5, U6, U7: moved to B.Cu
- C46, C47, C53, C58, C59: footprint Capacitor_SMD:C_01005_0402Metric -> Capacitor_SMD:C_0402_1005Metric; moved to B.Cu
- C95, U1: moved to F.Cu
- NT1: footprint NetTie:NetTie-2_SMD_Pad2.0mm -> NetTie:NetTie-2_SMD_Pad0.5mm; moved to B.Cu
- moved C62 152.5 mm to (157.9, 90.5), turned to -90 degrees
- moved R54 151.9 mm to (157.4, 95.2), turned to 180 degrees
- moved R56 150.7 mm to (157.4, 95.9), turned to 180 degrees
- moved R55 150.5 mm to (157.4, 93.7), turned to 180 degrees
- moved C48 150.0 mm to (157.1, 90.5), turned to -90 degrees
- moved C44 149.6 mm to (155.1, 87.6)
- moved C69 148.8 mm to (154.6, 90.5), turned to 90 degrees
- moved R53 148.8 mm to (157.4, 94.4), turned to 180 degrees
- moved R57 148.7 mm to (157.4, 93.0), turned to 180 degrees
- moved R52 148.6 mm to (157.4, 92.2), turned to 180 degrees
- moved C49 147.8 mm to (155.4, 90.5), turned to 90 degrees
- moved C43 145.8 mm to (148.5, 91.4), turned to 180 degrees
- moved R50 145.4 mm to (155.1, 85.8), turned to 180 degrees
- moved C42 144.5 mm to (148.5, 86.4), turned to 180 degrees
- moved R92 143.3 mm to (155.1, 87.0)
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Connections:
- C53 pad 1: /BLDC DRIVE3/BOOT1 -> /BLDC DRIVE/BOOT2
- C53 pad 2: /BLDC DRIVE3/A -> /BLDC DRIVE/B
- U12 pad 20: /SWDIO_M3 -> /STM32F051K8U7/SWDIO
- U12 pad 21: /SWCLK_M3 -> /STM32F051K8U7/SWCLK
- U13 pad 20: /SWDIO_M2 -> /STM32F051K8U9/SWDIO
- U13 pad 21: /SWCLK_M2 -> /STM32F051K8U9/SWCLK
- U6 pad 20: /SWDIO_M4 -> /STM32F051K8U6/SWDIO
- U6 pad 21: /SWCLK_M4 -> /STM32F051K8U6/SWCLK
- U7 pad 20: /SWDIO_M1 -> /STM32F051K8U8/SWDIO
- U7 pad 21: /SWCLK_M1 -> /STM32F051K8U8/SWCLK
Other:
- outline, holes or cut-outs redrawn
